Commit message: bugfix and warning suppress

File: tactile_sim/assets/embodiment_assets/combined_urdfs/mg400_flat_tactip.urdf (robot description, URDF)
Before this commit: robot mg400, 14 links, 13 joints
Joints:
- joint j5: axis -0.00001 0.00000 1.00000 -> 0.00000 0.00000 1.00000

File: tactile_sim/assets/embodiment_assets/combined_urdfs/mg400_mini_tactip.urdf (robot description, URDF)
Before this commit: robot mg400, 14 links, 13 joints
Joints:
- joint j5: axis -0.00001 0.00000 1.00000 -> 0.00000 0.00000 1.00000

File: tactile_sim/assets/embodiment_assets/combined_urdfs/mg400_right_angle_digit.urdf (robot description, URDF)
Before this commit: robot mg400, 14 links, 13 joints
Joints:
- joint j5: axis -0.00001 0.00000 1.00000 -> 0.00000 0.00000 1.00000

File: tactile_sim/assets/embodiment_assets/combined_urdfs/mg400_right_angle_digitac.urdf (robot description, URDF)
Before this commit: robot mg400, 14 links, 13 joints
Joints:
- joint j5: axis -0.00001 0.00000 1.00000 -> 0.00000 0.00000 1.00000

File: tactile_sim/assets/embodiment_assets/combined_urdfs/mg400_right_angle_tactip.urdf (robot description, URDF)
Before this commit: robot mg400, 15 links, 14 joints
Joints:
- joint j5: axis -0.00001 0.00000 1.00000 -> 0.00000 0.00000 1.00000

File: tactile_sim/assets/embodiment_assets/combined_urdfs/mg400_standard_digit.urdf (robot description, URDF)
Before this commit: robot mg400, 14 links, 13 joints
Joints:
- joint j5: axis -0.00001 0.00000 1.00000 -> 0.00000 0.00000 1.00000

File: tactile_sim/assets/embodiment_assets/combined_urdfs/mg400_standard_digitac.urdf (robot description, URDF)
Before this commit: robot mg400, 14 links, 13 joints
Joints:
- joint j5: axis -0.00001 0.00000 1.00000 -> 0.00000 0.00000 1.00000

File: tactile_sim/assets/embodiment_assets/combined_urdfs/mg400_standard_tactip.urdf (robot description, URDF)
Before this commit: robot mg400, 14 links, 13 joints
Joints:
- joint j5: axis -0.00001 0.00000 1.00000 -> 0.00000 0.00000 1.00000

File: tactile_sim/assets/robot_arm_assets/mg400/urdfs/mg400.urdf (robot description, URDF)
Before this commit: robot mg400, 11 links, 10 joints
Joints:
- joint j5: axis -1.19408295462994E-05 0 0.999999999928708 -> 0 0 1
